File: Izhitsa-a/Izhitsa-a.kicad_pcb (KiCad board)
At the start: 2 copper layers, 268.7 x 105.5 mm, 60 parts, among them J1 Conn_01x02, J2 Conn_01x02, J3 Conn_01x05, J5 USB_C_Receptacle_USB2.0, U1 STM32F072RBTx, U2 AMS1117-3.3

Commit message: Delete some element labels. Increase labels font size
Other:
- board text added: "3V3"
- board text removed: "+3V3"
